Commit message: a simple restruction of porject folder structure

File: urdf/mogi_bot/mogi_bot.urdf (robot description, URDF)
Before this commit: robot mogi_bot, 6 links, 5 joints
Links:
- link base_link: geometry collision box size=.4 .2 .1; collision sphere radius=0.0499
- link left_wheel: geometry collision cylinder length=.05 radius=.1; visual mesh filename=package://erl_assignment_1/urdf/mogi_bot/meshes/wheel.dae
- link right_wheel: geometry collision cylinder length=.05 radius=.1; visual mesh filename=package://erl_assignment_1/urdf/mogi_bot/meshes/wheel.dae

Commit message: modification

File: urdf/mogi_bot/mogi_bot.urdf (robot description, URDF)
Before this commit: robot mogi_bot, 6 links, 5 joints
Links:
- added link scan_link, mass 1e-5; collision box size=.1 .1 .1; visual mesh filename=package://erl_assignment_1/urdf/mogi_bot/meshes/lidar.dae
Joints:
- added joint scan_joint: type fixed, parent base_link, child scan_link, origin xyz=0 0 0.15 rpy=0 0 0
- joint camera_joint: origin xyz=0.225 0 0.075 rpy=0 0 0 -> xyz=0.225 0 0.075 rpy=0 0 0.785
